File: uk-01_mod/uk-01_mod.sch (KiCad schematic (older format))
At the start: 48 parts, among them J1 Conn_01x04_Male, J2 Conn_01x05_Male, J3 Conn_02x12_Counter_Clockwise, U1 SN74HC32N, U10 SN74HC32N, U11 SN74HC32N, U12 74HC595D_118, U13 SN74HC32N, U2 74HC595D_118, U3 SN74HC32N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

Commit message: 基板設計進めた
Parts:
- added J4: Conn_01x02_Male, symbol Connector:Conn_01x02_Male
Connections:
- net CON_DATA_1: now also U7.21 (GPA0); no longer U7.1 (GPB0)
- net CON_DATA_2: now also U7.22 (GPA1); no longer U7.2 (GPB1)
- net CON_DATA_3: now also U7.23 (GPA2); no longer U7.3 (GPB2)
- net CON_DATA_4: now also U7.24 (GPA3); no longer U7.4 (GPB3)
- net CON_DATA_5: now also U7.25 (GPA4); no longer U7.5 (GPB4)
- net CON_DATA_6: now also U7.26 (GPA5); no longer U7.6 (GPB5)
- net CON_DATA_7: now also U7.27 (GPA6); no longer U7.7 (GPB6)
- net CON_DATA_8: now also U7.28 (GPA7); no longer U7.8 (GPB7)
- net CON_SCAN_1: now also U7.1 (GPB0)
- net CON_SCAN_2: now also U7.2 (GPB1)
- net CON_SCAN_3: now also U7.3 (GPB2)
- net CON_SCAN_4: now also U7.4 (GPB3)
- net GND: now also J4.2 (Pin_2)
- new net PEDAL: J4.1 (Pin_1), U7.5 (GPB4)
- no-connect marks 5 -> 8
Other:
- moved on the sheet: J1, J2, J3, U12, U2, U5, U7, U9
